Commit message: Rebase from 'upstream'

File: models/example-robot-data/robots/kinova_description/robots/kinova.urdf (robot description, URDF)
Before this commit: robot kinova, 15 links, 14 joints
Links:
- removed link jaco_front_hatch_support_v2
- removed link jaco_mounting_block
Joints:
- removed joint base_to_jaco_support
- removed joint jaco_support_to_jaco_mounting_block
- joint jaco_mounting_block_to_j2s6s200_link_base: parent jaco_mounting_block -> base

File: models/example-robot-data/robots/panda_description/urdf/panda.urdf (robot description, URDF)
Before this commit: robot panda, 12 links, 11 joints
Links:
- added link panda_hand_tcp, mass 0
- link panda_hand: mass 0 -> 0.73
- link panda_leftfinger: mass 0 -> 0.015; geometry collision box size=17.5e-3 15.2e-3 18.5e-3; collision box size=17.5e-3 7e-3 23.5e-3
- link panda_link0: mass None -> 0.629769
- link panda_link1: mass 0 -> 4.970684
- link panda_link2: mass 0 -> 0.646926
- link panda_link3: mass 0 -> 3.228604
- link panda_link4: mass 0 -> 3.587895
- link panda_link5: mass 0 -> 1.225946
- link panda_link6: mass 0 -> 1.666555
- link panda_link7: mass 0 -> 0.735522
- link panda_rightfinger: mass 0 -> 0.015; geometry collision box size=17.5e-3 15.2e-3 18.5e-3; collision box size=17.5e-3 7e-3 23.5e-3
Joints:
- added joint panda_hand_tcp_joint: type fixed, parent panda_hand, child panda_hand_tcp, origin xyz=0 0 0.1034 rpy=0 0 0
- joint panda_finger_joint1: limit lower=0.0 upper=0.04 effort=20 velocity=0.2 -> lower=0.0 upper=0.04 effort=100 velocity=0.2
- joint panda_finger_joint2: limit lower=0.0 upper=0.04 effort=20 velocity=0.2 -> lower=0.0 upper=0.04 effort=100 velocity=0.2
- joint panda_hand_joint: origin xyz=0 0 0 rpy=0 0 -0.785398163397 -> xyz=0 0 0 rpy=0 0 -0.7853981633974483
- joint panda_joint1: limit lower=-2.9671 upper=2.9671 effort=87 velocity=2.3925 -> lower=-2.8973 upper=2.8973 effort=87.0 velocity=2.175
- joint panda_joint2: limit lower=-1.8326 upper=1.8326 effort=87 velocity=2.3925 -> lower=-1.7628 upper=1.7628 effort=87.0 velocity=2.175; origin xyz=0 0 0 rpy=-1.57079632679 0 0 -> xyz=0 0 0 rpy=-1.5707963267948966 0 0
- joint panda_joint3: limit lower=-2.9671 upper=2.9671 effort=87 velocity=2.3925 -> lower=-2.8973 upper=2.8973 effort=87.0 velocity=2.175; origin xyz=0 -0.316 0 rpy=1.57079632679 0 0 -> xyz=0 -0.316 0 rpy=1.5707963267948966 0 0
- joint panda_joint4: limit lower=-3.1416 upper=0.0873 effort=87 velocity=2.3925 -> lower=-3.0718 upper=-0.0698 effort=87.0 velocity=2.175; origin xyz=0.0825 0 0 rpy=1.57079632679 0 0 -> xyz=0.0825 0 0 rpy=1.5707963267948966 0 0
- joint panda_joint5: limit lower=-2.9671 upper=2.9671 effort=12 velocity=2.8710 -> lower=-2.8973 upper=2.8973 effort=12.0 velocity=2.61; origin xyz=-0.0825 0.384 0 rpy=-1.57079632679 0 0 -> xyz=-0.0825 0.384 0 rpy=-1.5707963267948966 0 0
- joint panda_joint6: limit lower=-0.0873 upper=3.8223 effort=12 velocity=2.8710 -> lower=-0.0175 upper=3.7525 effort=12.0 velocity=2.61; origin xyz=0 0 0 rpy=1.57079632679 0 0 -> xyz=0 0 0 rpy=1.5707963267948966 0 0
- joint panda_joint7: limit lower=-2.9671 upper=2.9671 effort=12 velocity=2.8710 -> lower=-2.8973 upper=2.8973 effort=12.0 velocity=2.61; origin xyz=0.088 0 0 rpy=1.57079632679 0 0 -> xyz=0.088 0 0 rpy=1.5707963267948966 0 0
- joint panda_joint8: axis 0 0 0 -> (none)
